Commit message: latest

File: scout_description/urdf/scout_mini.xacro (robot description, xacro)
@@ -1,5 +1,4 @@
 <?xml version="1.0"?>
-<robot name="scout_mini"
-    xmlns:xacro="http://ros.org/wiki/xacro">
+<robot name="scout_mini" xmlns:xacro="http://ros.org/wiki/xacro">
     <xacro:arg name="urdf_extras" default="scout_mini_extras.urdf" />
     <!-- Vehicle Geometries -->
@@ -7,17 +6,4 @@
     <xacro:property name="track" value="0.4563536" />
     <xacro:property name="wheel_vertical_offset" value="-0.077" />
-    <!-- For testing, hang the robot up in the air
-    <link name="world" />
-    <joint name="world_to_base_link" type="fixed">
-        <origin xyz="0 0 0.5" rpy="0 0 0" />
-        <parent link="world"/>
-        <child link="base_link"/>
-    </joint> -->
- <!-- <link name="base_footprint"/>
-  <joint name="base_joint" type="fixed">
-    <parent link="base_footprint"/>
-    <child link="base_link"/>
-    <origin xyz="0.0 0.0 0.010" rpy="0 0 0"/>
-  </joint> -->
     <!-- Base link -->
     <link name="base_link">
@@ -150,4 +136,48 @@
         <axis xyz="0 0 1" rpy="0 0 0" />
     </joint>
+    <!-- plug-in -->
+    <plugin name='scout_mini_joint_state' filename='libgazebo_ros_joint_state_publisher.so'>
+      <ros>
+        <namespace>/robot_namespace</namespace>
+        <remapping>~/out:=joint_states</remapping>
+      </ros>
+      <update_rate>50</update_rate>
+      <joint_name>front_right_wheel</joint_name>
+      <joint_name>front_left_wheel</joint_name>
+      <joint_name>rear_right_wheel</joint_name>
+      <joint_name>rear_left_wheel</joint_name>
+    </plugin>
+    <plugin name='skid_steer_drive' filename='libgazebo_ros_diff_drive.so'>
+      <!-- topics & remappings -->
+      <ros>
+        <namespace>/robot_namespace</namespace>
+        <remapping>/tf:=tf</remapping>
+      </ros>
+      <!-- Update rate -->
+      <update_rate>50</update_rate>
+      <!-- Number of wheel pairs -->
+      <num_wheel_pairs>2</num_wheel_pairs>
+      <!-- front wheels -->
+      <left_joint>front_left_wheel</left_joint>
+      <right_joint>front_right_wheel</right_joint>
+      <!-- rear wheels-->
+      <left_joint>rear_left_wheel</left_joint>
+      <right_joint>rear_right_wheel</right_joint>
+      <!-- kinematics -->
+      <wheel_separation>0.490</wheel_separation>
+      <wheel_separation>0.490</wheel_separation>
+      <wheel_diameter>0.160</wheel_diameter>
+      <wheel_diameter>0.160</wheel_diameter>
+      <!-- limits -->
+      <max_wheel_torque>20</max_wheel_torque>
+      <max_wheel_acceleration>1.0</max_wheel_acceleration>
+      <!-- output -->
+      <publish_odom>true</publish_odom>
+      <publish_odom_tf>true</publish_odom_tf>
+      <publish_wheel_tf>false</publish_wheel_tf>
+      <odometry_frame>odom</odometry_frame>
+      <odometry_topic>odom</odometry_topic>
+      <robot_base_frame>base_link</robot_base_frame>
+    </plugin>
     <!-- Additional definitions -->
     <xacro:include filename="$(arg urdf_extras)" />
